File: step_1/step_1/step_1.kicad_pcb (KiCad board)
At the start: 2 copper layers, 90 x 90 mm, 32 parts, among them J2 Conn_01x05_Pin, J3 Screw_Terminal_01x02, Q1 BC547, Q2 BC547, SW1 SW_SPDT, SW2 SW_SPDT, SW3 SW_SPDT, SW4 SW_Push, U1 SN74HC08N, U2 LM555xN, U3 74HC193, U4 CD74HC4511E, U5 HDSP-7803, U7 UA78M05QDCYRQ1

Commit message: all
Parts:
- added R8: 2.2k, Resistor_THT:R_Axial_DIN0207_L6.3mm_D2.5mm_P10.16mm_Horizontal, F.Cu at (138.4, 96.5)
- added R9: 2.2k, Resistor_THT:R_Axial_DIN0207_L6.3mm_D2.5mm_P10.16mm_Horizontal, F.Cu at (172.5, 142.0)
- moved R5 1.19 mm to (169.0, 142.1)
Connections:
- Q1 pad 2: /output -> Net-(Q1-B)
- Q2 pad 2: /output -> Net-(Q2-B)
Routing:
- net Net-(Q1-B): track 0.00 -> 8.54 mm
- net /output: track 114.7 -> 120.7 mm
- net Net-(Q2-B): track 0.00 -> 5.41 mm
