File: step_1/step_1/step_1.kicad_sch (KiCad schematic)
At the start: 35 parts, among them J1 Conn_01x06_Pin, J2 Conn_01x05_Pin, J3 Screw_Terminal_01x02, Q1 BC547, Q2 BC547, SW1 SW_SPDT, SW2 SW_SPDT, SW3 SW_SPDT, SW4 SW_Push, U1 SN74HC08N, U2 LM555xN, U3 74HC193, U4 CD74HC4511E, U5 HDSP-7803, U7 UA78M05QDCYRQ1

Commit message: all
Other:
- note added: "2 × NE555 (Steps 1 and 3) 2 × NE556, dual 555 timer (Steps 7 and 10 - one IC per step)"
- note removed: "2 × NE555 (Steps 1 and 3) 2 × 74HC123 (Steps 7 and 10 - one IC per step)"
Changed lines of the file:
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@@
 	(generator_version "10.0")
 	(paper "A4")
-	(text "2 × NE555    (Steps 1 and 3)\n2 × 74HC123  (Steps 7 and 10 - one IC per step)"
+	(text "2 × NE555    (Steps 1 and 3)\n2 × NE556, dual 555 timer  (Steps 7 and 10 - one IC per step)"
 		(exclude_from_sim no)
 		(at 21.59 176.784 0)

Commit message: all
Parts:
- C4: value 100nF -> 10nF; mouser 810-FG28X7R1H104KNT0 -> 594-K103K10X7RF53H5
Changed lines of the file:
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@@
 			)
 		)
-		(property "Value" "100nF"
+		(property "Value" "10nF"
 			(at 81.28 149.8599 0)
 			(show_name no)
@@
 			)
 		)
-		(property "mouser" "810-FG28X7R1H104KNT0 "
+		(property "mouser" "594-K103K10X7RF53H5"
 			(at 77.47 148.59 0)
 			(hide yes)
