File: step_10/step_10/step_10.kicad_sch (KiCad schematic)
At the start: 27 parts, among them J2 Conn_01x05_Pin, J3 Conn_01x05_Pin, Q1 BC547, Q2 BC547, SW1 SW_SPDT, SW2 SW_SPDT, U1 NE556, U2 SN74HC08N

Commit message: all
Parts:
- removed J3: Conn_01x05_Pin, Connector_PinHeader_2.54mm:PinHeader_1x05_P2.54mm_Horizontal, symbol Connector:Conn_01x05_Pin
Connections:
- net output_stp6 renamed output_stp9
